File: dual_loop_probe_0.2.kicad_pcb (KiCad board)
At the start: 4 copper layers, 99.5 x 33.5 mm, 11 parts, among them J1 Conn_Coaxial, J2 Conn_Coaxial

Commit message: update to version 0.2
Other:
- outline, holes or cut-outs redrawn
- board text added: "Rev. 0.2 2024-08-12"
- board text removed: "Rev. 0.1 2024-04-03"
Changed lines of the file:
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@@
 				(font
 					(size 1.27 1.27)
+					(thickness 0.15)
 				)
 			)
@@
 				(font
 					(size 1.27 1.27)
+					(thickness 0.15)
 				)
 			)
@@
 				(font
 					(size 1.27 1.27)
+					(thickness 0.15)
 				)
 			)
@@
 				(font
 					(size 1.27 1.27)
+					(thickness 0.15)
 				)
 			)
@@
 				(font
 					(size 1.27 1.27)
+					(thickness 0.15)
 				)
 			)
@@
 				(font
 					(size 1.27 1.27)
+					(thickness 0.15)
 				)
 			)
@@
 				(font
 					(size 1.27 1.27)
+					(thickness 0.15)
 				)
 			)
@@
 				(font
 					(size 1.27 1.27)
+					(thickness 0.15)
 				)
 			)
@@
 				(font
 					(size 1.27 1.27)
+					(thickness 0.15)
 				)
 			)
@@
 				(font
 					(size 1.27 1.27)
+					(thickness 0.15)
 				)
 			)
@@
 				(font
 					(size 1.27 1.27)
+					(thickness 0.15)
 				)
 			)
@@
 				(font
 					(size 1.27 1.27)
+					(thickness 0.15)
 				)
 			)
@@
 				(font
 					(size 1.27 1.27)
+					(thickness 0.15)
 				)
 			)
@@
 				(font
 					(size 1.27 1.27)
+					(thickness 0.15)
 				)
 			)
@@
 				(font
 					(size 1.27 1.27)
+					(thickness 0.15)
 				)
 			)
@@
 				(font
 					(size 1.27 1.27)
+					(thickness 0.15)
 				)
 			)
@@
 				(font
 					(size 1.27 1.27)
+					(thickness 0.15)
 				)
 			)
@@
 				(font
 					(size 1.27 1.27)
+					(thickness 0.15)
 				)
 			)
@@
 				(font
 					(size 1.27 1.27)
+					(thickness 0.15)
 				)
 			)
@@
 				(font
 					(size 1.27 1.27)
+					(thickness 0.15)
 				)
 			)
@@
 				(font
 					(size 1.27 1.27)
+					(thickness 0.15)
 				)
 			)
@@
 				(font
 					(size 1.27 1.27)
+					(thickness 0.15)
 				)
 			)
@@
 				(font
 					(size 1.27 1.27)
+					(thickness 0.15)
 				)
 			)
@@
 				(font
 					(size 1.27 1.27)
+					(thickness 0.15)
 				)
 			)
@@
 				(font
 					(size 1.27 1.27)
+					(thickness 0.15)
 				)
 			)
@@
 				(font
 					(size 1.27 1.27)
+					(thickness 0.15)
 				)
 			)
@@
 				(font
 					(size 1.27 1.27)
+					(thickness 0.15)
 				)
 			)
@@
 				(font
 					(size 1.27 1.27)
+					(thickness 0.15)
 				)
 			)
@@
 				(font
 					(size 1.27 1.27)
+					(thickness 0.15)
 				)
 			)
@@
 				(font
 					(size 1.27 1.27)
+					(thickness 0.15)
 				)
 			)
@@
 				(font
 					(size 1.27 1.27)
+					(thickness 0.15)
 				)
 			)
@@
 				(font
 					(size 1.27 1.27)
+					(thickness 0.15)
 				)
 			)
@@
 				(font
 					(size 1.27 1.27)
+					(thickness 0.15)
 				)
 			)
@@
 	(gr_poly
 		(pts
-			(xy 171 93.499081) (xy 171 94.499081) (xy 174 94.499081) (xy 174 93.499081)
+			(xy 171 93.5) (xy 171 94.5) (xy 174 94.5) (xy 174 93.5)
 		)
 		(stroke
@@
 		(layer "Edge.Cuts")
 	)
-	(gr_arc
-		(start 184.75 90.75)
-		(mid 181 92.022954)
-		(end 177.25 90.75)
-		(stroke
-			(width 0.15)
-			(type default)
-		)
-		(layer "Edge.Cuts")
-	)
 	(gr_line
 		(start 192.5 85)
@@
 		(layer "Edge.Cuts")
 	)
-	(gr_arc
-		(start 177.25 90.75)
-		(mid 181 89.477046)
-		(end 184.75 90.75)
-		(stroke
-			(width 0.15)
-			(type default)
-		)
-		(layer "Edge.Cuts")
-	)
 	(gr_line
 		(start 181 107.5)
@@
 		)
 	)
-	(gr_text "Rev. 0.1  2024-04-03"
+	(gr_text "Rev. 0.2  2024-08-12"
 		(at 141 104.5 0)
 		(layer "F.SilkS")
@@
 			(pts
 				(xy 175 108) (xy 169 99.5) (xy 100 99.5) (xy 98 101.5) (xy 93 101.5) (xy 93 97.5) (xy 98.5 97.5)
-				(xy 98.5 94.5) (xy 93 94.5) (xy 93 90.5) (xy 98 90.60519) (xy 100 92.5) (xy 169 92.5) (xy 170.5 90.5)
-				(xy 183 90.5) (xy 184 91) (xy 185 91) (xy 187 92.5) (xy 187 94.5) (xy 186.5 95.5) (xy 187 95.5)
+				(xy 98.5 94.5) (xy 93 94.5) (xy 93 90.5) (xy 98 90.5) (xy 100 92.5) (xy 169 92.5) (xy 170.5 90.5)
+				(xy 183 90.5) (xy 184 90.5) (xy 185 90.5) (xy 187 92.5) (xy 187 94.5) (xy 186.5 95.5) (xy 187 95.5)
 				(xy 188.5 94) (xy 192.5 92.5) (xy 192.5 108)
 			)
@@
 		(polygon
 			(pts
-				(xy 184 90.5) (xy 183 91) (xy 170.5 91) (xy 169 89) (xy 100 89) (xy 98 91) (xy 93 91) (xy 93 87)
-				(xy 98.5 87) (xy 98.5 84) (xy 93 84) (xy 93 80) (xy 98 80.10519) (xy 100 82) (xy 169 82) (xy 175 73.5)
-				(xy 192.5 73.5) (xy 192.5 85) (xy 192.5 89) (xy 188.5 87.5) (xy 187 86) (xy 186.5 86) (xy 187 87)
-				(xy 187 89) (xy 185 90.5)
-			)
-		)
-	)
-	(zone
-		(net 1)
-		(net_name "GND")
-		(layer "In1.Cu")
-		(name "top GND")
-		(hatch edge 0.508)
-		(connect_pads yes
-			(clearance 0.6)
-		)
-		(min_thickness 0.254)
-		(filled_areas_thickness no)
-		(fill yes
-			(thermal_gap 0.508)
-			(thermal_bridge_width 0.508)
-			(smoothing fillet)
-			(radius 0.5)
-		)
-		(polygon
-			(pts
-				(xy 170.5 91) (xy 169 89) (xy 100 89) (xy 98 91) (xy 93 91) (xy 93 87) (xy 98.5 87) (xy 98.5 84)
-				(xy 93 84) (xy 93 80) (xy 98 80.10519) (xy 100 82) (xy 169 82) (xy 175 73.5) (xy 192.5 73.5) (xy 192.5 85)
-				(xy 192.5 89) (xy 187 86) (xy 184.5 91)
+				(xy 184 91) (xy 183 91) (xy 170.5 91) (xy 169 89) (xy 100 89) (xy 98 91) (xy 93 91) (xy 93 87) (xy 98.5 87)
+				(xy 98.5 84) (xy 93 84) (xy 93 80) (xy 98 80) (xy 100 82) (xy 169 82) (xy 175 73.5) (xy 192.5 73.5)
+				(xy 192.5 85) (xy 192.5 89) (xy 188.5 87.5) (xy 187 86) (xy 186.5 86) (xy 187 87) (xy 187 89) (xy 185 91)
 			)
 		)
